File: s2k_kpro.brd (EAGLE design)
At the start: 69.8 x 25.4 mm, 74 parts, among them IC1 LMV321ILT, IC2 MAX9926, IC3 AD5175BRMZ, IC5 MKE02Z16LVC, IC6 74LVC1G17SE, IC7 74LVC2G32DP, X1 12MHz

Commit message: Final review, sent for manufacturing.
Parts:
- removed C14: 47uF, resistor:D/7343-31R
- removed R18: 10k, resistor:R0603
- removed R19: 270, resistor:R0603
- added C20: 10uF, resistor:C0603
- added R4: 2.2k, resistor:R0603
- added R8: 100, resistor:R0603
- C1: value 10uF -> 10pF; device resistor:C0805 -> resistor:C0603
- C10: value 10uF -> 1uF; device resistor:C0805 -> resistor:C0603
- C12: device resistor:C0603 -> resistor:C0805
- C2: value 0.1uF -> 10pF
- C3: value 10pF -> 10uF; device resistor:C0603 -> resistor:C0805
- C4: value 10pF -> 0.1uF
- C6: value 10uF -> 10nF; device resistor:C0805 -> parts:C0306
- C8: value 10nF -> 10uF; device parts:C0306 -> resistor:C0805
- C9: value 1uF -> 47uF; device resistor:C0603 -> resistor:D/7343-31R
- R11: value 10k -> 0
- R12: value 0 -> 100
- R14: value 10k -> 100
- R15, R25: value 100 -> 10k
- R16: value 100 -> 270
- R21: value 0 -> 1k
- R22: value 1k -> 0
- R23: value 10k -> 1k
- R24: value 2.2k -> 10k
- R26: value 1k -> 10k
- moved R25 42.5 mm to (14.0, 15.9), flipped to the bottom, turned to 90 degrees
- moved R15 38.4 mm to (55.9, 12.7), turned to 0 degrees
- moved C12 36.7 mm to (55.9, 2.54), flipped to the top, turned to 180 degrees
- moved C9 30.9 mm to (27.7, 22.9)
- moved R23 29.8 mm to (26.7, 15.9), turned to 270 degrees
- moved R26 29.8 mm to (55.9, 10.2), turned to 0 degrees
- moved R11 21.7 mm to (45.7, 14.0), flipped to the top, turned to 180 degrees
- moved R24 16.2 mm to (24.1, 15.9), flipped to the bottom, turned to 90 degrees
- moved R13 12.3 mm to (55.9, 21.0), turned to 0 degrees
- moved R16 10.0 mm to (55.9, 7.62)
- moved R2 8.91 mm to (34.9, 3.81)
- moved C4 8.64 mm to (38.7, 3.81), turned to 270 degrees
- moved C10 7.62 mm to (55.9, 10.2), turned to 0 degrees
- moved C6 7.62 mm to (15.2, 14.0)
- moved C8 7.62 mm to (15.2, 21.6)
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- renumbered C13 to C21, C15 to C23, C16 to C22, R17 to R27
Connections:
- removed net N$17: CKP.TP, R25.2
- new net ECT_OUT: DASH.TP, R5.2
- net +5V: now also C12.1, C3.2, C4.2, C9.+, R15.2, R4.1; no longer C1.2, C10.1, C14.+, C2.2, R14.2, R2.1
- net CAM_IN+: now also CM+.TP, IC2.16; no longer CK+.TP, IC2.10
- net CAM_IN-: now also CM-.TP, IC2.15; no longer CK-.TP, IC2.9
- net CAM_OUT: now also R12.2; no longer R16.2
- net CAM_TDC: now also R11.2; no longer R13.2
- net CRANK_IN+: now also CK+.TP, IC2.9; no longer CM+.TP, IC2.16
- net CRANK_IN-: now also CK-.TP, IC2.10; no longer CM-.TP, IC2.15
- net CRANK_OUT: now also CKP.TP, R14.2; no longer DASH.TP, R15.2
- net ECT_SENSE: now also U$1.6; no longer U$1.5
- net EXTAL: now also C2.1; no longer C3.1
- net GND: now also C1.2, C2.2, C20.2, C3.1, C4.1, C9.-, R13.2, R25.2, R26.2; no longer C1.1, C14.-, C2.1, C3.2, C4.2, C9.2, R12.2, R18.2, R23.2
- net LED_B: now also R8.2; no longer R5.2
- net LED_G: now also R7.2; no longer R6.2
- net LED_R: now also R6.2; no longer R7.2
- net N$1: now also IC7.7, R12.1; no longer IC7.3, R16.1
- net N$10: now also R22.1; no longer R21.1
- net N$11: now also R13.1; no longer R12.1
- net N$12: now also R7.1; no longer R6.1
- net N$13: now also R8.1; no longer R5.1
- net N$14: now also IC7.3, R14.1; no longer IC7.7, R25.1
- net N$15: now also R23.2, R24.1; no longer R11.1, R26.2
- net N$16: now also R5.1; no longer R15.1
- net N$18: now also R25.1; no longer R18.1
- net N$27: now also C10.1; no longer C9.1
- net N$28: now also R16.1, R26.1; no longer R19.1, R23.1
- net N$29: now also R16.2; no longer R19.2
- net N$3: now also R4.2; no longer R2.2
- net N$4: now also R2.1, U$1.5; no longer R24.1, U$1.6
- net N$6: now also R11.1; no longer R13.1
- net N$7: now also R2.2; no longer R24.2
- net N$8: now also R24.2; no longer R11.2
- net N$9: now also R6.1; no longer R7.1
- net NRST: now also R15.1; no longer R14.1
- net THR_PWM: now also R23.1; no longer R26.1
- net VR_BIAS: now also C20.1, R21.1; no longer C12.1, R22.1
- net XTAL: now also C1.1; no longer C4.1
Routing:
- net GND: track 92.6 -> 80.2 mm, vias 6 -> 5
- net N$17: track 10.8 -> 0.00 mm
- net ECT_OUT: track 0.00 -> 9.67 mm
- net CAM_IN+: track 24.7 -> 18.2 mm
- net CAM_IN-: track 17.1 -> 12.8 mm
- net CRANK_IN-: track 12.8 -> 17.0 mm
- net CRANK_IN+: track 18.2 -> 22.1 mm
- net N$4: track 4.83 -> 3.59 mm
- net CRANK_OUT: track 9.67 -> 10.6 mm
- net ECT_SENSE: track 14.2 -> 13.3 mm
- net CAM_OUT: track 5.86 -> 5.02 mm
- net N$1: track 5.92 -> 6.65 mm
- net IAT_SENSE: track 15.2 -> 15.9 mm
- net CMP_EDGE: track 12.4 -> 12.9 mm
Other:
- board text added: "5V"
- board text added: "CTS"
- board text added: "Copyright Owen Kirby 9/11/2016"
- board text added: "DTR"
- board text added: "RX"
- board text added: "TX"
