File: s2k_kpro.sch (EAGLE design)
At the start: 74 parts, among them IC1 LMV321ILT, IC2 MAX9926, IC3 AD5175BRMZ, IC5 MKE02Z16LVC, IC6 74LVC1G17SE, IC7 74LVC2G32DP, X1 12MHz

Commit message: Final review, sent for manufacturing.
Parts:
- removed C14: 47uF, resistor:CPOL-USD/7343-31R
- removed R18: 10k, resistor:R-US_R0603
- removed R19: 270, resistor:R-US_R0603
- added C20: 10uF, resistor:C-USC0603
- added R4: 2.2k, resistor:R-US_R0603
- added R8: 100, resistor:R-US_R0603
- C1: value 10uF -> 10pF; device resistor:C-USC0805 -> resistor:C-USC0603
- C10: value 10uF -> 1uF; device resistor:C-USC0805 -> resistor:C-USC0603
- C12: device resistor:C-USC0603 -> resistor:C-USC0805; DNP DNP -> (none)
- C2: value 0.1uF -> 10pF
- C3: value 10pF -> 10uF; device resistor:C-USC0603 -> resistor:C-USC0805
- C4: value 10pF -> 0.1uF
- C6: value 10uF -> 10nF; device resistor:C-USC0805 -> parts:CAP-0306
- C8: value 10nF -> 10uF; device parts:CAP-0306 -> resistor:C-USC0805
- C9: value 1uF -> 47uF; device resistor:C-USC0603 -> resistor:CPOL-USD/7343-31R
- R10: DNP DNP -> (none)
- R11: value 10k -> 0
- R12: value 0 -> 100
- R14: value 10k -> 100
- R15: value 100 -> 10k
- R16: value 100 -> 270
- R21: value 0 -> 1k
- R22: value 1k -> 0
- R23: value 10k -> 1k; DNP DNP -> (none)
- R24: value 2.2k -> 10k
- R25: value 100 -> 10k; DNP (none) -> DNP
- R26: value 1k -> 10k; DNP (none) -> DNP
- renumbered C13 to C21, C15 to C23, C16 to C22, R17 to R27
Connections:
- removed net N$17: CKP.P, R25.2
- new net ECT_OUT: DASH.P, R5.2
- net +5V: now also C12.1, C3.2, C4.2, C9.+, R15.2, R4.1; no longer C1.2, C10.1, C14.+, C2.2, R14.2, R2.1
- net CAM_IN+: now also CM+.P, IC2.IN1+; no longer CK+.P, IC2.IN2-
- net CAM_IN-: now also CM-.P, IC2.IN1-; no longer CK-.P, IC2.IN2+
- net CAM_OUT: now also R12.2; no longer R16.2
- net CAM_TDC: now also R11.2; no longer R13.2
- net CRANK_IN+: now also CK+.P, IC2.IN2+; no longer CM+.P, IC2.IN1+
- net CRANK_IN-: now also CK-.P, IC2.IN2-; no longer CM-.P, IC2.IN1-
- net CRANK_OUT: now also CKP.P, R14.2; no longer DASH.P, R15.2
- net EXTAL: now also C2.1; no longer C3.1
- net GND: now also C1.2, C2.2, C20.2, C3.1, C4.1, C9.-, R13.2, R25.2, R26.2; no longer C1.1, C14.-, C2.1, C3.2, C4.2, C9.2, R12.2, R18.2, R23.2
- net LED_B: now also R8.2; no longer R5.2
- net LED_G: now also R7.2; no longer R6.2
- net LED_R: now also R6.2; no longer R7.2
- net N$1: now also R12.1; no longer R16.1
- net N$10: now also R22.1; no longer R21.1
- net N$11: now also R13.1; no longer R12.1
- net N$12: now also R7.1; no longer R6.1
- net N$13: now also R8.1; no longer R5.1
- net N$14: now also R14.1; no longer R25.1
- net N$15: now also R23.2, R24.1; no longer R11.1, R26.2
- net N$16: now also R5.1; no longer R15.1
- net N$18: now also R25.1; no longer R18.1
- net N$27: now also C10.1; no longer C9.1
- net N$28: now also R16.1, R26.1; no longer R19.1, R23.1
- net N$29: now also R16.2; no longer R19.2
- net N$3: now also R4.2; no longer R2.2
- net N$4: now also R2.1; no longer R24.1
- net N$6: now also R11.1; no longer R13.1
- net N$7: now also R2.2; no longer R24.2
- net N$8: now also R24.2; no longer R11.2
- net N$9: now also R6.1; no longer R7.1
- net NRST: now also R15.1; no longer R14.1
- net THR_PWM: now also R23.1; no longer R26.1
- net VR_BIAS: now also C20.1, R21.1; no longer C12.1, R22.1
- net XTAL: now also C1.1; no longer C4.1
Other:
- moved on the sheet: C1, C10, C12, C2, C3, C4, C6, C8, CK+, CK-, LED1, R12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
